File: panelX_MEGA/Lnet.kicad_sch (KiCad schematic)
At the start: 11 parts, among them J501 RJ12, Q501 AO3400A, U501 LM311

Commit message: added nano project to repo. Must be modular flatcable design. I want to make 2 versions, one with voltage regulator and Xnet and one as I2C slave
Parts:
- J501: footprint (none) -> Connector_RJ:RJ12_Amphenol_54601
Changed lines of the file:
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@@
     (property "Reference" "J501" (id 0) (at 64.77 71.12 0))
     (property "Value" "RJ12" (id 1) (at 72.39 71.12 0))
-    (property "Footprint" "" (id 2) (at 69.85 81.915 90)
+    (property "Footprint" "Connector_RJ:RJ12_Amphenol_54601" (id 2) (at 69.85 81.915 90)
       (effects (font (size 1.27 1.27)) hide)
     )
