File: panelX_MEGA/MEGA.kicad_sch (KiCad schematic)
At the start: 2 parts

Commit message: added nano project to repo. Must be modular flatcable design. I want to make 2 versions, one with voltage regulator and Xnet and one as I2C slave
Parts:
- U201: value (none) -> WeMos_D1_mini; footprint (none) -> Module:WEMOS_D1_mini_light
- XA201: footprint (none) -> Arduino:Arduino_Mega2560_Shield
Connections:
- net dir: now also XA201.A0; no longer XA201.D53 (D53_SS)
- no-connect marks 25 -> 46
Changed lines of the file:
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@@
   (no_connect (at 41.91 74.93))
   (no_connect (at 90.17 67.31))
+  (no_connect (at 90.17 82.55))
+  (no_connect (at 90.17 85.09))
+  (no_connect (at 90.17 87.63))
+  (no_connect (at 90.17 90.17))
+  (no_connect (at 90.17 92.71))
+  (no_connect (at 90.17 95.25))
+  (no_connect (at 156.21 146.05))
+  (no_connect (at 156.21 148.59))
+  (no_connect (at 156.21 151.13))
+  (no_connect (at 156.21 153.67))
+  (no_connect (at 156.21 156.21))
+  (no_connect (at 156.21 143.51))
+  (no_connect (at 90.17 110.49))
+  (no_connect (at 90.17 113.03))
+  (no_connect (at 90.17 115.57))
+  (no_connect (at 90.17 118.11))
+  (no_connect (at 90.17 97.79))
+  (no_connect (at 90.17 100.33))
+  (no_connect (at 90.17 102.87))
+  (no_connect (at 90.17 105.41))
+  (no_connect (at 90.17 107.95))
   (no_connect (at 90.17 49.53))
   (no_connect (at 90.17 46.99))
@@
     (stroke (width 0) (type default) (color 0 0 0 0))
   )
-  (wire (pts (xy 156.21 156.21) (xy 165.1 156.21))
+  (wire (pts (xy 90.17 80.01) (xy 81.28 80.01))
     (stroke (width 0) (type default) (color 0 0 0 0))
   )
@@
     )
   )
-  (global_label "dir" (shape input) (at 165.1 156.21 0) (fields_autoplaced)
-    (effects (font (size 1.27 1.27)) (justify left))
-    (property "Intersheet References" "${INTERSHEET_REFS}" (id 0) (at 170.0531 156.2894 0)
-      (effects (font (size 1.27 1.27)) (justify left) hide)
+  (global_label "dir" (shape input) (at 81.28 80.01 180) (fields_autoplaced)
+    (effects (font (size 1.27 1.27)) (justify right))
+    (property "Intersheet References" "${INTERSHEET_REFS}" (id 0) (at 76.3269 79.9306 0)
+      (effects (font (size 1.27 1.27)) (justify right) hide)
     )
   )
@@
       (effects (font (size 1.27 1.27)) (justify right))
     )
-    (property "Value" "" (id 1) (at 52.5906 87.1173 0)
+    (property "Value" "WeMos_D1_mini" (id 1) (at 52.5906 87.1173 0)
       (effects (font (size 1.27 1.27)) (justify right))
     )
-    (property "Footprint" "" (id 2) (at 52.07 93.98 0)
+    (property "Footprint" "Module:WEMOS_D1_mini_light" (id 2) (at 52.07 93.98 0)
       (effects (font (size 1.27 1.27)) hide)
     )
@@
       (effects (font (size 1.524 1.524)))
     )
-    (property "Footprint" "" (id 2) (at 140.97 31.75 0)
+    (property "Footprint" "Arduino:Arduino_Mega2560_Shield" (id 2) (at 140.97 31.75 0)
       (effects (font (size 1.524 1.524)) hide)
     )
@@
       (effects (font (size 1.27 1.27)) hide)
     )
-    (property "Value" "" (id 1) (at 52.07 92.0734 0))
+    (property "Value" "GND" (id 1) (at 52.07 92.0734 0))
     (property "Footprint" "" (id 2) (at 52.07 87.63 0)
       (effects (font (size 1.27 1.27)) hide)
