File: panelX_MEGA/flatcable.kicad_sch (KiCad schematic)
At the start: 1 part

Commit message: added nano project to repo. Must be modular flatcable design. I want to make 2 versions, one with voltage regulator and Xnet and one as I2C slave
Parts:
- J401: value (none) -> Conn_02x20_Counter_Clockwise
Changed lines of the file:
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@@
     (in_bom yes) (on_board yes)
     (property "Reference" "J401" (id 0) (at 142.24 55.9902 0))
-    (property "Value" "" (id 1) (at 146.05 48.26 0))
+    (property "Value" "Conn_02x20_Counter_Clockwise" (id 1) (at 146.05 48.26 0))
     (property "Footprint" "" (id 2) (at 140.97 83.82 0)
       (effects (font (size 1.27 1.27)) hide)
