File: panelX_MEGA/panelX_MEGA.kicad_pcb (KiCad board)
At the start: 2 copper layers, 101.1 x 55.7 mm, 26 parts, among them J301 RJ12, J401 Conn_02x20_Counter_Clockwise, J501 RJ12, Q501 AO3400A, U201 WeMos_D1_mini, U301 MAX485E, U501 LM311, U601 24LC256

Commit message: added nano project to repo. Must be modular flatcable design. I want to make 2 versions, one with voltage regulator and Xnet and one as I2C slave
Parts:
- J401: footprint Connector_PinHeader_2.54mm:PinHeader_2x20_P2.54mm_Vertical_SMD -> Connector_PinHeader_2.54mm:PinHeader_2x20_P2.54mm_Vertical
- moved J401 24.4 mm to (157.2, 111.8)
Connections:
- U201 pad 9: +5C -> +5V
- XA201 pad A0: unconnected-(XA201-PadA0) -> dir
- XA201 pad D53: dir -> unconnected-(XA201-PadD53)
Routing:
- net +5V: track 15.9 -> 176.7 mm, vias 0 -> 6
- net Tx: track 2.88 -> 77.8 mm, vias 0 -> 1
- net +12V: track 3.81 -> 75.5 mm, vias 0 -> 2
- net Rx: track 2.88 -> 72.3 mm, vias 0 -> 1
- net Lnet_Tx: track 2.27 -> 59.1 mm, vias 0 -> 1
- net Lnet_Rx: track 4.23 -> 49.1 mm, vias 0 -> 1
- net dir: track 5.49 -> 48.5 mm
- net /Xnet/B: track 3.01 -> 13.1 mm
- net /Xnet/A: track 3.01 -> 11.0 mm
- net Net-(D301-Pad2): track 0.00 -> 7.84 mm
- net GPIO3: track 46.3 -> 53.9 mm
- net GPIO5: track 42.0 -> 49.6 mm
- net GPIO7: track 38.5 -> 46.0 mm
- net GPIO1: track 49.6 -> 56.3 mm
- net GPIO4: track 49.2 -> 54.7 mm
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