File: PanelX_NANO/EEPROM.kicad_sch (KiCad schematic)
At the start: 7 parts

Commit message: Deleted zip files from repo
Parts:
- C501: value (none) -> 100nF; footprint (none) -> Capacitor_SMD:C_0603_1608Metric_Pad1.08x0.95mm_HandSolder
- JP501, JP503: footprint (none) -> Jumper:SolderJumper-3_P1.3mm_Bridged12_RoundedPad1.0x1.5mm_NumberLabels
- JP502: value (none) -> SolderJumper_3_Bridged12; footprint (none) -> Jumper:SolderJumper-3_P1.3mm_Bridged12_RoundedPad1.0x1.5mm_NumberLabels
- R501, R502: value (none) -> 4k7; footprint (none) -> Resistor_SMD:R_0603_1608Metric
- U501: value (none) -> 24LC256; footprint (none) -> Package_SO:SOIC-8_3.9x4.9mm_P1.27mm
Changed lines of the file:
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@@
       (effects (font (size 1.27 1.27)) (justify left))
     )
-    (property "Value" "" (id 1) (at 168.3894 99.1671 0)
+    (property "Value" "24LC256" (id 1) (at 168.3894 99.1671 0)
       (effects (font (size 1.27 1.27)) (justify left))
     )
-    (property "Footprint" "" (id 2) (at 166.37 105.41 0)
+    (property "Footprint" "Package_SO:SOIC-8_3.9x4.9mm_P1.27mm" (id 2) (at 166.37 105.41 0)
       (effects (font (size 1.27 1.27)) hide)
     )
@@
       (effects (font (size 1.27 1.27)) (justify left) hide)
     )
-    (property "Footprint" "" (id 2) (at 118.11 114.3 0)
+    (property "Footprint" "Jumper:SolderJumper-3_P1.3mm_Bridged12_RoundedPad1.0x1.5mm_NumberLabels" (id 2) (at 118.11 114.3 0)
       (effects (font (size 1.27 1.27)) hide)
     )
@@
       (effects (font (size 1.27 1.27)) hide)
     )
-    (property "Value" "" (id 1) (at 166.37 123.8234 0))
+    (property "Value" "GND" (id 1) (at 166.37 123.8234 0))
     (property "Footprint" "" (id 2) (at 166.37 119.38 0)
       (effects (font (size 1.27 1.27)) hide)
@@
       (effects (font (size 1.27 1.27)) (justify left))
     )
-    (property "Value" "" (id 1) (at 183.388 99.4922 0)
+    (property "Value" "4k7" (id 1) (at 183.388 99.4922 0)
       (effects (font (size 1.27 1.27)) (justify left))
     )
-    (property "Footprint" "" (id 2) (at 179.832 97.79 90)
+    (property "Footprint" "Resistor_SMD:R_0603_1608Metric" (id 2) (at 179.832 97.79 90)
       (effects (font (size 1.27 1.27)) hide)
     )
@@
       (effects (font (size 1.27 1.27)) hide)
     )
-    (property "Value" "" (id 1) (at 123.19 123.8234 0))
+    (property "Value" "GND" (id 1) (at 123.19 123.8234 0))
     (property "Footprint" "" (id 2) (at 123.19 119.38 0)
       (effects (font (size 1.27 1.27)) hide)
@@
       (effects (font (size 1.27 1.27)) (justify left))
     )
-    (property "Value" "" (id 1) (at 192.278 99.4922 0)
+    (property "Value" "4k7" (id 1) (at 192.278 99.4922 0)
       (effects (font (size 1.27 1.27)) (justify left))
     )
-    (property "Footprint" "" (id 2) (at 188.722 97.79 90)
+    (property "Footprint" "Resistor_SMD:R_0603_1608Metric" (id 2) (at 188.722 97.79 90)
       (effects (font (size 1.27 1.27)) hide)
     )
@@
       (effects (font (size 1.27 1.27)) (justify left) hide)
     )
-    (property "Footprint" "" (id 2) (at 118.11 91.44 0)
+    (property "Footprint" "Jumper:SolderJumper-3_P1.3mm_Bridged12_RoundedPad1.0x1.5mm_NumberLabels" (id 2) (at 118.11 91.44 0)
       (effects (font (size 1.27 1.27)) hide)
     )
@@
       (effects (font (size 1.27 1.27)) (justify right))
     )
-    (property "Value" "" (id 1) (at 141.859 105.8422 0)
+    (property "Value" "100nF" (id 1) (at 141.859 105.8422 0)
       (effects (font (size 1.27 1.27)) (justify right))
     )
-    (property "Footprint" "" (id 2) (at 145.7452 100.33 0)
+    (property "Footprint" "Capacitor_SMD:C_0603_1608Metric_Pad1.08x0.95mm_HandSolder" (id 2) (at 145.7452 100.33 0)
       (effects (font (size 1.27 1.27)) hide)
     )
@@
       (effects (font (size 1.27 1.27)) (justify left))
     )
-    (property "Value" "" (id 1) (at 119.8122 104.5209 90)
+    (property "Value" "SolderJumper_3_Bridged12" (id 1) (at 119.8122 104.5209 90)
       (effects (font (size 1.27 1.27)) (justify left) hide)
     )
-    (property "Footprint" "" (id 2) (at 118.11 102.87 0)
+    (property "Footprint" "Jumper:SolderJumper-3_P1.3mm_Bridged12_RoundedPad1.0x1.5mm_NumberLabels" (id 2) (at 118.11 102.87 0)
       (effects (font (size 1.27 1.27)) hide)
     )
@@
       (effects (font (size 1.27 1.27)) hide)
     )
-    (property "Value" "" (id 1) (at 166.37 87.8642 0))
+    (property "Value" "+5V" (id 1) (at 166.37 87.8642 0))
     (property "Footprint" "" (id 2) (at 166.37 91.44 0)
       (effects (font (size 1.27 1.27)) hide)

Commit message: I picked a suitable connector. I will use plain 2x12 female n male connectors for the b2b connector. Death to flatcables! The RJ12 connector still goed on the panel carrier board. I will look for vertical SMD variant
Parts:
- renumbered C501 to C2, JP501 to JP1, JP502 to JP2, JP503 to JP3, R501 to R5, R502 to R6, U501 to U2
Changed lines of the file:
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@@
   (symbol (lib_id "Memory_EEPROM:24LC256") (at 166.37 105.41 0) (unit 1)
     (in_bom yes) (on_board yes) (fields_autoplaced)
-    (property "Reference" "U501" (id 0) (at 168.3894 96.6302 0)
+    (property "Reference" "U2" (id 0) (at 168.3894 96.6302 0)
       (effects (font (size 1.27 1.27)) (justify left))
     )
@@
   (symbol (lib_id "Jumper:SolderJumper_3_Bridged12") (at 118.11 114.3 180) (unit 1)
     (in_bom yes) (on_board yes)
-    (property "Reference" "JP503" (id 0) (at 118.11 116.84 0)
+    (property "Reference" "JP3" (id 0) (at 118.11 116.84 0)
       (effects (font (size 1.27 1.27)) (justify left))
     )
@@
   (symbol (lib_id "power:GND") (at 166.37 119.38 0) (unit 1)
     (in_bom yes) (on_board yes) (fields_autoplaced)
-    (property "Reference" "#PWR0504" (id 0) (at 166.37 125.73 0)
+    (property "Reference" "#PWR09" (id 0) (at 166.37 125.73 0)
       (effects (font (size 1.27 1.27)) hide)
     )
@@
   (symbol (lib_id "Device:R") (at 181.61 97.79 0) (unit 1)
     (in_bom yes) (on_board yes) (fields_autoplaced)
-    (property "Reference" "R501" (id 0) (at 183.388 96.9553 0)
+    (property "Reference" "R5" (id 0) (at 183.388 96.9553 0)
       (effects (font (size 1.27 1.27)) (justify left))
     )
@@
   (symbol (lib_id "power:GND") (at 123.19 119.38 0) (unit 1)
     (in_bom yes) (on_board yes) (fields_autoplaced)
-    (property "Reference" "#PWR0503" (id 0) (at 123.19 125.73 0)
+    (property "Reference" "#PWR08" (id 0) (at 123.19 125.73 0)
       (effects (font (size 1.27 1.27)) hide)
     )
@@
   (symbol (lib_id "Device:R") (at 190.5 97.79 0) (unit 1)
     (in_bom yes) (on_board yes) (fields_autoplaced)
-    (property "Reference" "R502" (id 0) (at 192.278 96.9553 0)
+    (property "Reference" "R6" (id 0) (at 192.278 96.9553 0)
       (effects (font (size 1.27 1.27)) (justify left))
     )
@@
   (symbol (lib_id "Jumper:SolderJumper_3_Bridged12") (at 118.11 91.44 180) (unit 1)
     (in_bom yes) (on_board yes)
-    (property "Reference" "JP501" (id 0) (at 117.475 94.615 0)
+    (property "Reference" "JP1" (id 0) (at 117.475 94.615 0)
       (effects (font (size 1.27 1.27)) (justify left))
     )
@@
   (symbol (lib_id "Device:C") (at 144.78 104.14 0) (mirror x) (unit 1)
     (in_bom yes) (on_board yes) (fields_autoplaced)
-    (property "Reference" "C501" (id 0) (at 141.859 103.3053 0)
+    (property "Reference" "C2" (id 0) (at 141.859 103.3053 0)
       (effects (font (size 1.27 1.27)) (justify right))
     )
@@
   (symbol (lib_id "power:+5V") (at 113.03 87.63 0) (unit 1)
     (in_bom yes) (on_board yes) (fields_autoplaced)
-    (property "Reference" "#PWR0501" (id 0) (at 113.03 91.44 0)
+    (property "Reference" "#PWR06" (id 0) (at 113.03 91.44 0)
       (effects (font (size 1.27 1.27)) hide)
     )
@@
   (symbol (lib_id "Jumper:SolderJumper_3_Bridged12") (at 118.11 102.87 180) (unit 1)
     (in_bom yes) (on_board yes)
-    (property "Reference" "JP502" (id 0) (at 118.11 105.41 0)
+    (property "Reference" "JP2" (id 0) (at 118.11 105.41 0)
       (effects (font (size 1.27 1.27)) (justify left))
     )
@@
   (symbol (lib_id "power:+5V") (at 166.37 91.44 0) (unit 1)
     (in_bom yes) (on_board yes) (fields_autoplaced)
-    (property "Reference" "#PWR0502" (id 0) (at 166.37 95.25 0)
+    (property "Reference" "#PWR07" (id 0) (at 166.37 95.25 0)
       (effects (font (size 1.27 1.27)) hide)
     )
